File: FPGA.kicad_sch (KiCad schematic)
At the start: 9 parts, among them J4 Conn_01x06_Pin, U2 a, U3 W25Q32JVSS, Y2 ASE-xxxMHz

Commit message: Added more I/O. Changed power regulators
Parts:
- added R40: 2.2k, symbol Device:R
Connections:
- net A10_AP is gone; now on net DQ5: U2.E2 (IOL_10A)
- net A12_BC_B is gone; now on net DQ3: U2.F1 (IOL_12A)
- net BA0 is gone; now on net DQ0: U2.F3 (IOL_13B_GBIN7)
- net BA1 is gone; now on net CLK: U2.G1 (IOL_14A_GBIN6)
- net CK is gone; now on net A3: U2.E11 (IOR_148)
- net CK_B is gone; now on net A2: U2.D11 (IOR_152)
- net ODT is gone; now on net A0: U2.C11 (IOR_160)
- net RST_B is gone; now on net A1: U2.D10 (IOR_154)
- net A0: no longer U2.B1 (IOL_2A)
- net A1: no longer U2.B2 (IOL_2B)
- net A11: now also U2.G11 (IOR_129); no longer U2.E3 (IOL_10B)
- net A14: now also U2.H11 (IOR_119); no longer U2.F4 (IOL_13A)
- net A2: no longer U2.C4 (IOL_4A)
- net A3: no longer U2.C3 (IOL_4B)
- net A4: now also U2.D9 (IOR_147); no longer U2.C2 (IOL_5A)
- net A5: now also U2.E8 (IOR_146); no longer U2.C1 (IOL_5B)
- net A6: now also U2.E9 (IOR_144); no longer U2.E1 (IOL_8A)
- net A7: now also U2.E10 (IOR_141_GBIN2); no longer U2.D1 (IOL_8B)
- net A8: now also U2.F11 (IOR_140_GBIN3); no longer U2.D2 (IOL_9A)
- net A9: now also U2.F9 (IOR_137); no longer U2.D3 (IOL_9B)
- net DQ0: no longer U2.J11 (IOR_114)
- net DQ1: now also U2.F4 (IOL_13A); no longer U2.K11 (IOR_115)
- net DQ10: now also U2.C1 (IOL_5B); no longer U2.F9 (IOR_137)
- net DQ11: now also U2.C2 (IOL_5A); no longer U2.F11 (IOR_140_GBIN3)
- net DQ12: now also U2.C3 (IOL_4B); no longer U2.E10 (IOR_141_GBIN2)
- net DQ13: now also U2.C4 (IOL_4A); no longer U2.E9 (IOR_144)
- net DQ14: now also U2.B2 (IOL_2B); no longer U2.E8 (IOR_146)
- net DQ15: now also U2.B1 (IOL_2A); no longer U2.D9 (IOR_147)
- net DQ2: now also U2.F2 (IOL_12B); no longer U2.H10 (IOR_116)
- net DQ3: no longer U2.J10 (IOR_117)
- net DQ4: now also U2.E3 (IOL_10B); no longer U2.G8 (IOR_118)
- net DQ5: no longer U2.H11 (IOR_119)
- net DQ6: now also U2.D3 (IOL_9B); no longer U2.G10 (IOR_120)
- net DQ7: now also U2.D2 (IOL_9A); no longer U2.G9 (IOR_128)
- net DQ8: now also U2.D1 (IOL_8B); no longer U2.G11 (IOR_129)
- net DQ9: now also U2.E1 (IOL_8A); no longer U2.F10 (IOR_136)
- net P3V3: now also R40.2
- net IO_B7: now reaches U2.A2 (IOT_222)
- net IO_B13: now reaches U2.H7 (IOB_87)
- net IO_B8: now reaches U2.H9 (IOB_104_CBSEL1)
- net SRAM_WE_B: now reaches U2.J3 (IOB_57)
- net SRAM_UB_B: now reaches U2.J4 (IOB_64)
- net IO_B18: now reaches U2.J5 (IOB_78)
- net IO_B14: now reaches U2.J7 (IOB_86)
- net IO_B11: now reaches U2.J8 (IOB_91)
- net SRAM_CE2: now reaches U2.K3 (IOB_63)
- net IO_B19: now reaches U2.K4 (IOB_73)
- net IO_B17: now reaches U2.K5 (IOB_79)
- net IO_B15: now reaches U2.K6 (IOB_82_GBIN4)
- net IO_B12: now reaches U2.K7 (IOB_89)
- net CDONE: now reaches U2.K8 (CDONE)
- net CDONE: now also R40.1
- net SRAM_OE_B: now reaches U2.L1 (IOB_56)
- net SRAM_CE_B: now reaches U2.L2 (IOB_61)
- net SRAM_LB_B: now reaches U2.L3 (IOB_71)
- net IO_B20: now reaches U2.L4 (IOB_72)
- net IO_B16: now reaches U2.L5 (IOB_81_GBIN5)
- net IO_B10: now reaches U2.L7 (IOB_94)
- net IO_B9: now reaches U2.L8 (IOB_103_CBSEL0)
- net BA2 renamed IO_B3
- net CAS_B renamed USB1_DN
- net CKE renamed IO_B4
- net CS_B renamed IO_B2
- net IO_1 renamed IO_T1
- net IO_10 renamed IO_T10
- net IO_2 renamed IO_T2
- net IO_3 renamed IO_T3
- net IO_4 renamed IO_T4
- net IO_5 renamed IO_T5
- net IO_6 renamed IO_T6
- net IO_7 renamed IO_T7
- net IO_8 renamed IO_T8
- net IO_9 renamed IO_T9
- net LDM renamed IO_B6
- net LDQS renamed USB2_DN
- net LDQS_B renamed USB2_DP
- net P1V1 renamed P1V2
- net RAS_B renamed IO_B1
- net UDM renamed IO_B5
- net UDQS renamed USB3_DN
- net UDQS_B renamed USB3_DP
- net WE_B renamed USB1_DP
- new net A10: U2.F10 (IOR_136)
- new net A12: U2.G9 (IOR_128)
- new net A13: U2.G10 (IOR_120)
- new net A15: U2.G8 (IOR_118)
- new net A16: U2.J10 (IOR_117)
- new net A17: U2.H10 (IOR_116)
- new net A18: U2.K11 (IOR_115)
- new net A19: U2.J11 (IOR_114)
- no-connect marks 3 -> 2

Commit message: Power routed. Saving before reworking ICE40 pins to optimize layout
Parts:
- added JP2: Jumper_2_Small_Open, Button_Switch_SMD:SW_DIP_SPSTx01_Slide_6.7x4.1mm_W6.73mm_P2.54mm_LowProfile_JPin, symbol Jumper:Jumper_2_Small_Open
- added R36: 4.7k, Resistor_SMD:R_0603_1608Metric, symbol Device:R
- C14: footprint (none) -> Capacitor_SMD:C_0603_1608Metric
- J4: footprint (none) -> Connector_PinHeader_2.54mm:PinHeader_1x06_P2.54mm_Vertical
- R16, R17, R18, R22, R40: footprint (none) -> Resistor_SMD:R_0603_1608Metric
Connections:
- net IO_B20 is gone; now on net IO_B6: U2.L4 (IOB_72)
- net USB1_DN is gone; now on net IO_B2: U2.H1 (IOL_18A)
- net USB1_DP is gone; now on net IO_B1: U2.H2 (IOL_18B)
- net USB_DN is gone; now on net LED_G: U2.B4 (IOT_219)
- net USR_BTN is gone; now on net LED_R: U2.D5 (IOT_212)
- net IO_B1: no longer U2.H3 (IOL_17B)
- net IO_B10: now also U2.A2 (IOT_222); no longer U2.L7 (IOB_94)
- net IO_B2: no longer U2.G3 (IOL_17A)
- net IO_B3: now also U2.H3 (IOL_17B); no longer U2.G2 (IOL_14B)
- net IO_B4: now also U2.G3 (IOL_17A); no longer U2.B11 (IOR_161)
- net IO_B5: now also U2.G2 (IOL_14B); no longer U2.A1 (IOT_225)
- net IO_B6: no longer U2.A3 (IOT_223)
- net IO_B7: now also U2.B11 (IOR_161); no longer U2.A2 (IOT_222)
- net IO_B8: now also U2.A1 (IOT_225); no longer U2.H9 (IOB_104_CBSEL1)
- net IO_B9: now also U2.A3 (IOT_223); no longer U2.L8 (IOB_103_CBSEL0)
- net IO_T1: now also U2.B5 (IOT_208); no longer U2.A6 (IOT_206)
- net IO_T10: now also U2.C8 (IOT_179); no longer U2.B8 (IOT_177)
- net IO_T2: now also U2.A5 (IOT_207); no longer U2.B6 (IOT_198_GBIN0)
- net IO_T3: now also U2.A6 (IOT_206); no longer U2.B7 (IOT_197_GBIN1)
- net IO_T4: now also U2.B6 (IOT_198_GBIN0); no longer U2.A7 (IOT_192)
- net IO_T5: now also U2.B7 (IOT_197_GBIN1); no longer U2.C7 (IOT_191)
- net IO_T6: now also U2.A7 (IOT_192); no longer U2.A8 (IOT_190)
- net IO_T7: now also U2.C7 (IOT_191); no longer U2.D7 (IOT_181)
- net IO_T8: now also U2.A8 (IOT_190); no longer U2.C8 (IOT_179)
- net IO_T9: now also U2.D7 (IOT_181); no longer U2.A9 (IOT_178)
- net LED_B: now also U2.A4 (IOT_211); no longer U2.A5 (IOT_207)
- net LED_G: no longer U2.A4 (IOT_211)
- net LED_R: no longer U2.B5 (IOT_208)
- net P3V3: now also R36.2
- net SPI_CNFG_CS_B: now also JP2.1 (A); no longer J4.1 (Pin_1), R16.1, U2.K10 (IOB_108_SS), U3.1 (~{CS})
- net SPI_CNFG_SCK: now also R16.1
- net CRESET_B: now reaches R22.1, U2.L9 (~{CRESET})
- net F: now reaches U2.B10 (VPP_FAST)
- net IO_B11 renamed FIFO_RXF_B
- net IO_B12 renamed FIFO7
- net IO_B13 renamed FIFO6
- net IO_B14 renamed FIFO5
- net IO_B15 renamed FIFO4
- net IO_B16 renamed FIFO3
- net IO_B17 renamed FIFO2
- net IO_B18 renamed FIFO1
- net IO_B19 renamed FIFO0
- net SD_CS renamed SD_DAT3
- net SD_MISO renamed SD_DAT0
- net SD_MOSI renamed SD_DAT1
- net SD_SCK renamed SD_DAT2
- net SPI_CNFG_SDI renamed SPI_CNFG_DI
- net SPI_CNFG_SDO renamed SPI_CNFG_DO
- net USB_DP renamed USR_BTN1
- new net FIFO_RD_B: U2.L8 (IOB_103_CBSEL0)
- new net FIFO_TXE_B: U2.L7 (IOB_94)
- new net FIFO_WR_B: U2.H9 (IOB_104_CBSEL1)
- new net SD_CLK: U2.A9 (IOT_178)
- new net SD_CMD: U2.B8 (IOT_177)
- new net SPI_CNFG_CS: J4.1 (Pin_1), JP2.2 (B), R36.1, U2.K10 (IOB_108_SS), U3.1 (~{CS})
Other:
- note added: "DPair"
- moved on the sheet: J4, R16, R17, R18, U3

Commit message: Finished board. Added BOM
Connections:
- net A0: now also U2.L7 (IOB_94); no longer U2.C11 (IOR_160)
- net A1: now also U2.L8 (IOB_103_CBSEL0); no longer U2.D10 (IOR_154)
- net A10: now also U2.B11 (IOR_161); no longer U2.F10 (IOR_136)
- net A11: now also U2.B9 (IOT_174); no longer U2.G11 (IOR_129)
- net A12: now also U2.A11 (IOT_168); no longer U2.G9 (IOR_128)
- net A13: now also U2.A10 (IOT_170); no longer U2.G10 (IOR_120)
- net A14: now also U2.A9 (IOT_178); no longer U2.H11 (IOR_119)
- net A15: now also U2.A8 (IOT_190); no longer U2.G8 (IOR_118)
- net A16: now also U2.A5 (IOT_207); no longer U2.J10 (IOR_117)
- net A17: now also U2.G11 (IOR_129); no longer U2.H10 (IOR_116)
- net A18: now also U2.F10 (IOR_136); no longer U2.K11 (IOR_115)
- net A19: now also U2.D10 (IOR_154); no longer U2.J11 (IOR_114)
- net A2: now also U2.K11 (IOR_115); no longer U2.D11 (IOR_152)
- net A3: now also U2.J10 (IOR_117); no longer U2.E11 (IOR_148)
- net A4: now also U2.J11 (IOR_114); no longer U2.D9 (IOR_147)
- net A5: now also U2.H10 (IOR_116); no longer U2.E8 (IOR_146)
- net A6: now also U2.H11 (IOR_119); no longer U2.E9 (IOR_144)
- net A7: now also U2.G10 (IOR_120); no longer U2.E10 (IOR_141_GBIN2)
- net A8: now also U2.C11 (IOR_160); no longer U2.F11 (IOR_140_GBIN3)
- net A9: now also U2.C9 (IOT_172); no longer U2.F9 (IOR_137)
- net DQ0: now also U2.J8 (IOB_91); no longer U2.F3 (IOL_13B_GBIN7)
- net DQ1: now also U2.H9 (IOB_104_CBSEL1); no longer U2.F4 (IOL_13A)
- net DQ10: now also U2.F9 (IOR_137); no longer U2.C1 (IOL_5B)
- net DQ11: now also U2.E9 (IOR_144); no longer U2.C2 (IOL_5A)
- net DQ12: now also U2.D7 (IOT_181); no longer U2.C3 (IOL_4B)
- net DQ13: now also U2.C7 (IOT_191); no longer U2.C4 (IOL_4A)
- net DQ14: now also U2.B7 (IOT_197_GBIN1); no longer U2.B2 (IOL_2B)
- net DQ15: now also U2.A6 (IOT_206); no longer U2.B1 (IOL_2A)
- net DQ2: now also U2.G9 (IOR_128); no longer U2.F2 (IOL_12B)
- net DQ3: now also U2.E8 (IOR_146); no longer U2.F1 (IOL_12A)
- net DQ4: now also U2.D9 (IOR_147); no longer U2.E3 (IOL_10B)
- net DQ5: now also U2.C8 (IOT_179); no longer U2.E2 (IOL_10A)
- net DQ6: now also U2.B8 (IOT_177); no longer U2.D3 (IOL_9B)
- net DQ7: now also U2.A7 (IOT_192); no longer U2.D2 (IOL_9A)
- net DQ8: now also U2.H7 (IOB_87); no longer U2.D1 (IOL_8B)
- net DQ9: now also U2.G8 (IOR_118); no longer U2.E1 (IOL_8A)
- net FIFO0: now also U2.H1 (IOL_18A); no longer U2.K4 (IOB_73)
- net FIFO1: now also U2.H2 (IOL_18B); no longer U2.J5 (IOB_78)
- net FIFO2: now also U2.G2 (IOL_14B); no longer U2.K5 (IOB_79)
- net FIFO3: now also U2.F1 (IOL_12A); no longer U2.L5 (IOB_81_GBIN5)
- net FIFO4: now also U2.F2 (IOL_12B); no longer U2.K6 (IOB_82_GBIN4)
- net FIFO5: now also U2.E1 (IOL_8A); no longer U2.J7 (IOB_86)
- net FIFO6: now also U2.E2 (IOL_10A); no longer U2.H7 (IOB_87)
- net FIFO7: now also U2.D1 (IOL_8B); no longer U2.K7 (IOB_89)
- net FIFO_RD_B: now also U2.J5 (IOB_78); no longer U2.L8 (IOB_103_CBSEL0)
- net FIFO_RXF_B: now also U2.D2 (IOL_9A); no longer U2.J8 (IOB_91)
- net FIFO_TXE_B: now also U2.H3 (IOL_17B); no longer U2.L7 (IOB_94)
- net FIFO_WR_B: now also U2.J1 (IOL_23A); no longer U2.H9 (IOB_104_CBSEL1)
- net IO_B1: now also U2.K6 (IOB_82_GBIN4); no longer U2.H2 (IOL_18B)
- net IO_B10: now also U2.L1 (IOB_56); no longer U2.A2 (IOT_222)
- net IO_B2: now also U2.K5 (IOB_79); no longer U2.H1 (IOL_18A)
- net IO_B3: now also U2.L5 (IOB_81_GBIN5); no longer U2.H3 (IOL_17B)
- net IO_B4: now also U2.K4 (IOB_73); no longer U2.G3 (IOL_17A)
- net IO_B5: now also U2.L4 (IOB_72); no longer U2.G2 (IOL_14B)
- net IO_B6: now also U2.K3 (IOB_63); no longer U2.L4 (IOB_72)
- net IO_B7: now also U2.L3 (IOB_71); no longer U2.B11 (IOR_161)
- net IO_B8: now also U2.K2 (IOL_25A); no longer U2.A1 (IOT_225)
- net IO_B9: now also U2.L2 (IOB_61); no longer U2.A3 (IOT_223)
- net IO_T1: now also U2.B6 (IOT_198_GBIN0); no longer U2.B5 (IOT_208)
- net IO_T10: now also U2.C1 (IOL_5B); no longer U2.C8 (IOT_179)
- net IO_T2: now also U2.B5 (IOT_208); no longer U2.A5 (IOT_207)
- net IO_T3: now also U2.A4 (IOT_211); no longer U2.A6 (IOT_206)
- net IO_T4: now also U2.B4 (IOT_219); no longer U2.B6 (IOT_198_GBIN0)
- net IO_T5: now also U2.A3 (IOT_223); no longer U2.B7 (IOT_197_GBIN1)
- net IO_T6: now also U2.B3 (IOT_221); no longer U2.A7 (IOT_192)
- net IO_T7: now also U2.A2 (IOT_222); no longer U2.C7 (IOT_191)
- net IO_T8: now also U2.C2 (IOL_5A); no longer U2.A8 (IOT_190)
- net IO_T9: now also U2.A1 (IOT_225); no longer U2.D7 (IOT_181)
- net LED_B: now also U2.K1 (IOL_23B); no longer U2.A4 (IOT_211)
- net LED_G: now also U2.J3 (IOB_57); no longer U2.B4 (IOT_219)
- net LED_R: now also U2.J2 (IOL_25B); no longer U2.D5 (IOT_212)
- net SD_CLK: now also U2.E3 (IOL_10B); no longer U2.A9 (IOT_178)
- net SD_CMD: now also U2.F4 (IOL_13A); no longer U2.B8 (IOT_177)
- net SD_DAT0: now also U2.D3 (IOL_9B); no longer U2.B9 (IOT_174)
- net SD_DAT1: now also U2.D5 (IOT_212); no longer U2.C9 (IOT_172)
- net SD_DAT2: now also U2.G3 (IOL_17A); no longer U2.A10 (IOT_170)
- net SD_DAT3: now also U2.F3 (IOL_13B_GBIN7); no longer U2.A11 (IOT_168)
- net SRAM_CE2: now also U2.E11 (IOR_148); no longer U2.K3 (IOB_63)
- net SRAM_CE_B: now also U2.K7 (IOB_89); no longer U2.L2 (IOB_61)
- net SRAM_LB_B: now also U2.F11 (IOR_140_GBIN3); no longer U2.L3 (IOB_71)
- net SRAM_OE_B: now also U2.J7 (IOB_86); no longer U2.L1 (IOB_56)
- net SRAM_UB_B: now also U2.E10 (IOR_141_GBIN2); no longer U2.J4 (IOB_64)
- net SRAM_WE_B: now also U2.D11 (IOR_152); no longer U2.J3 (IOB_57)
- net USB2_DN: now also U2.B1 (IOL_2A); no longer U2.J1 (IOL_23A)
- net USB2_DP: now also U2.B2 (IOL_2B); no longer U2.K1 (IOL_23B)
- net USB3_DN: now also U2.C4 (IOL_4A); no longer U2.K2 (IOL_25A)
- net USB3_DP: now also U2.C3 (IOL_4B); no longer U2.J2 (IOL_25B)
- net USR_BTN1: now also U2.J4 (IOB_64); no longer U2.B3 (IOT_221)
Other:
- moved on the sheet: U2E

Commit message: End of Version 1.0. Feedback received
Other:
- note added: "PWR + CNFG |---------|"
- note removed: "POWER + CNFG |---------|"
- moved on the sheet: C14, J4, JP2, R16, R17, R18, R22, R36, R40, U2A, U2B, U2C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
