File: hardware/rev2.0/SeedSBC_rev2_0.kicad_pcb (KiCad board)
At the start: 8 copper layers, 86.4 x 53.3 mm, 156 parts, among them J1 Conn_01x12_Pin, J2 Micro_SD_Card, J3 Conn_01x02_Pin, J4 Conn_01x06_Pin, J6 USB_C_Receptacle_USB2.0_16P, J7 USB_C_Receptacle_USB2.0_16P, J8 Conn_01x14_Pin, Q2 BSS84, SW1 SW_Push, U1 TLV62568DBV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

Commit message: Fixed ReadMe. Fixed PCB Silkscreen
Other:
- board text added: "CHG"
- board text added: "PGOOD"
Changed lines of the file:
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@@
 		(tags "mountinghole M2")
 		(property "Reference" "H1"
-			(at 0 -3.15 0)
+			(at 0 -2.78 0)
 			(layer "F.SilkS")
 			(effects
 				(font
-					(size 1 1)
-					(thickness 0.15)
+					(size 0.5 0.5)
+					(thickness 0.125)
 				)
 			)
@@
 		(tags "mountinghole M2")
 		(property "Reference" "H2"
-			(at 0 -3.15 0)
+			(at 0 -2.78 0)
 			(layer "F.SilkS")
 			(effects
 				(font
-					(size 1 1)
-					(thickness 0.15)
+					(size 0.5 0.5)
+					(thickness 0.125)
 				)
 			)
@@
 		(tags "LED")
 		(property "Reference" "D6"
-			(at 2 -0.91 0)
+			(at 3.75 -0.9 0)
 			(layer "F.SilkS")
 			(effects
@@
 		(tags "mountinghole M2")
 		(property "Reference" "H3"
-			(at 0 -3.15 0)
+			(at 0 2.84 0)
 			(layer "F.SilkS")
 			(effects
 				(font
-					(size 1 1)
-					(thickness 0.15)
+					(size 0.5 0.5)
+					(thickness 0.125)
 				)
 			)
@@
 		(tags "mountinghole M2")
 		(property "Reference" "H4"
-			(at 0 -3.15 0)
+			(at 0 2.85 0)
 			(layer "F.SilkS")
 			(effects
 				(font
-					(size 1 1)
-					(thickness 0.15)
+					(size 0.5 0.5)
+					(thickness 0.125)
 				)
 			)
@@
 		(tags "LED")
 		(property "Reference" "D2"
-			(at 1.9775 -0.94 0)
+			(at 4.6875 -0.94 0)
 			(layer "F.SilkS")
 			(effects
@@
 		)
 	)
+	(gr_text "CHG"
+		(at 105.94 105.76 0)
+		(layer "F.SilkS")
+		(effects
+			(font
+				(size 0.5 0.5)
+				(thickness 0.125)
+				(bold yes)
+			)
+			(justify left bottom)
+		)
+	)
 	(gr_text "DI"
 		(at 155.22 123.03 90)
@@
 		)
 	)
+	(gr_text "PGOOD"
+		(at 105 104.37 0)
+		(layer "F.SilkS")
+		(effects
+			(font
+				(size 0.5 0.5)
+				(thickness 0.125)
+				(bold yes)
+			)
+			(justify left bottom)
+		)
+	)
